Commit message: Starts ARIAC2019, arms are not working

File: ur5_vel_start/urdf/ur5.urdf.xacro (robot description, xacro)
@@ -71,5 +71,5 @@
     </inertial>
   </xacro:macro>
-  <xacro:macro name="ur5_robot" params="prefix joint_limited">
+  <xacro:macro name="ur10" params="prefix joint_limited">
     <link name="${prefix}base_link" >
       <visual>

File: ur5_vel_start/urdf/ur5_robot.urdf.xacro (robot description, xacro)
@@ -1,5 +1,5 @@
 <?xml version="1.0"?>
 <robot xmlns:xacro="http://www.ros.org/wiki/xacro"
-       name="ur5_robot" >
+       name="ur10" >
   <xacro:property name="PI" value="3.14159265359"/>
   <xacro:property name="flange_radius" value="0.04"/>
@@ -18,5 +18,5 @@
   <xacro:include filename="$(find ur5_vel_start)/urdf/ur5.urdf.xacro" />
   <!-- arm -->
-  <xacro:ur5_robot prefix="$(arg ns)" joint_limited="true"/>
+  <xacro:ur10 prefix="$(arg ns)" joint_limited="true"/>
   <link name="world" />
   <joint name="world_joint" type="fixed">
